Commit message: Added Lidar Sensor on the Robot

File: description/lidar.xacro (robot description, xacro)
@@ -24,4 +24,5 @@
     <!-- LASER FRAME -->
     <gazebo reference="laser_frame">
+        <material>Gazebo/Red</material>
         <sensor name="laser" type="ray">
             <pose>0 0 0 0 0 0</pose>
